File: hardware/rs485_interface_boards/rs485_interface_board_RevA/_autosave-rs485_interface_board_RevA.kicad_sch (KiCad schematic)
At the start: 5 parts, among them J1 615006141121, J3 Conn_01x03, U1 SN65HVD3082EP

Commit message: completed rs-485 eth rev a board, generated pcb
Parts:
- added C1, C2: 100 nf, Capacitor_SMD:C_0805_2012Metric, symbol Device:C
- added R1, R2: 10k, Resistor_THT:R_Axial_DIN0207_L6.3mm_D2.5mm_P7.62mm_Horizontal, symbol Device:R
- added R3, R4: 10 Ohm, Resistor_SMD:R_0603_1608Metric, symbol Device:R
- added U2: SM712.TCT, footprints:SOT23_SEM, symbol TVS:SM712.TCT
- renumbered J3 to J1, J1 to J2
Connections:
- net +5V: now also C1.2, C2.1, R1.1
- net GND: now also C1.1, C2.2, R2.2, U2.3; no longer U1.2 (*RE)
- net at J2.1: now also R3.2, U2.2
- net at J2.2: now also R4.2, U2.1
- net at J1.3 (Pin_3), U1.1 (R): now also R1.2
- net at J1.2 (Pin_2), U1.3 (DE): now also U1.2 (*RE), R2.1
Other:
- moved on the sheet: 5V1, GND1, J1, U1
